File: nt-980/nt980.kicad_sch (KiCad schematic)
At the start: 225 parts, among them J1 USB, J2 ISP, K1 KEYSW, K10 KEYSW, K100 KEYSW, K101 KEYSW, K102 KEYSW, K103 KEYSW, K104 KEYSW, K105 KEYSW, K106 KEYSW, K107 KEYSW, K11 KEYSW, K12 KEYSW, K13 KEYSW, K14 KEYSW, K15 KEYSW, K16 KEYSW, K17 KEYSW, K18 KEYSW, K19 KEYSW, K20 KEYSW, K21 KEYSW, K22 KEYSW, K23 KEYSW, K24 KEYSW, K25 KEYSW, K26 KEYSW, K27 KEYSW, K28 KEYSW, K29 KEYSW, K3 KEYSW, K30 KEYSW, K31 KEYSW, K32 KEYSW, K33 KEYSW, K34 KEYSW, K35 KEYSW, K36 KEYSW, K37 KEYSW, K38 KEYSW, K39 KEYSW, K4 KEYSW, K40 KEYSW, K41 KEYSW, K42 KEYSW, K43 KEYSW, K44 KEYSW, K45 KEYSW, K46 KEYSW, K47 KEYSW, K48 KEYSW, K49 KEYSW, K5 KEYSW, K50 KEYSW, K51 KEYSW, K52 KEYSW, K53 KEYSW, K54 KEYSW, K55 KEYSW, K56 KEYSW, K57 KEYSW, K58 KEYSW, K59 KEYSW, K6 KEYSW, K60 KEYSW, K61 KEYSW, K62 KEYSW, K63 KEYSW, K64 KEYSW, K65 KEYSW, K66 KEYSW, K67 KEYSW, K68 KEYSW, K68-1 KEYSW, K69 KEYSW, K7 KEYSW, K70 KEYSW, K71 KEYSW, K73 KEYSW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

Commit message: add new files
Parts:
- added D2: D, Keeb_components:D_0805, symbol Device:D_ALT
- added K2: KEYSW, Connector_PinHeader_2.54mm:PinHeader_1x01_P2.54mm_Vertical, symbol keyboard_parts:KEYSW
Connections:
- net SCK: now also D2.1 (K)
- net col0: now also K2.2
- new net: D2.2 (A), K2.1

Commit message: add udb jst
Parts:
- added J3: UDB, Connector_JST:JST_SH_SM04B-SRSS-TB_1x04-1MP_P1.00mm_Horizontal, symbol Connector_Generic:Conn_01x04
Connections:
- net D+: now also J3.3 (Pin_3)
- net D-: now also J3.2 (Pin_2)
- net GND: now also J3.4 (Pin_4)
- net VUSB: now also J3.1 (Pin_1)
Changed lines of the file:
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@@
   (junction (at 156.21 215.9) (diameter 1.016) (color 0 0 0 0))
   (junction (at 156.21 232.41) (diameter 1.016) (color 0 0 0 0))
+  (junction (at 157.48 86.36) (diameter 1.016) (color 0 0 0 0))
   (junction (at 160.02 43.18) (diameter 1.016) (color 0 0 0 0))
   (junction (at 160.02 50.8) (diameter 1.016) (color 0 0 0 0))
@@
     (stroke (width 0) (type solid) (color 0 0 0 0))
   )
+  (wire (pts (xy 157.48 91.44) (xy 157.48 86.36))
+    (stroke (width 0) (type solid) (color 0 0 0 0))
+  )
   (wire (pts (xy 157.48 129.54) (xy 156.21 129.54))
     (stroke (width 0) (type solid) (color 0 0 0 0))
@@
     )
   )
+  (global_label "D-" (shape input) (at 157.48 93.98 180)
+    (effects (font (size 0.9906 0.9906)) (justify right))
+    (property "Intersheet References" "${INTERSHEET_REFS}" (id 0) (at 240.03 -58.42 0)
+      (effects (font (size 1.27 1.27)) hide)
+    )
+  )
+  (global_label "D+" (shape input) (at 157.48 96.52 180)
+    (effects (font (size 0.9906 0.9906)) (justify right))
+    (property "Intersheet References" "${INTERSHEET_REFS}" (id 0) (at 240.03 -53.34 0)
+      (effects (font (size 1.27 1.27)) hide)
+    )
+  )
   (global_label "col3" (shape input) (at 172.72 120.65 90)
     (effects (font (size 0.9906 0.9906)) (justify left))
@@
     (pin "1")
   )
+  (symbol (lib_id "power:GND") (at 157.48 99.06 0) (unit 1)
+    (in_bom yes) (on_board yes) (fields_autoplaced)
+    (property "Reference" "#PWR0122" (id 0) (at 157.48 105.41 0)
+      (effects (font (size 1.27 1.27)) hide)
+    )
+    (property "Value" "GND" (id 1) (at 157.48 104.14 0))
+    (property "Footprint" "" (id 2) (at 157.48 99.06 0)
+      (effects (font (size 1.27 1.27)) hide)
+    )
+    (property "Datasheet" "" (id 3) (at 157.48 99.06 0)
+      (effects (font (size 1.27 1.27)) hide)
+    )
+    (pin "1")
+  )
   (symbol (lib_id "Power:GND") (at 204.47 46.99 270) (unit 1)
     (in_bom yes) (on_board yes)
@@
     (pin "2")
   )
+  (symbol (lib_id "Connector_Generic:Conn_01x04") (at 162.56 93.98 0) (unit 1)
+    (in_bom yes) (on_board yes) (fields_autoplaced)
+    (property "Reference" "J3" (id 0) (at 165.1 93.9799 0)
+      (effects (font (size 1.27 1.27)) (justify left))
+    )
+    (property "Value" "UDB" (id 1) (at 165.1 96.5199 0)
+      (effects (font (size 1.27 1.27)) (justify left))
+    )
+    (property "Footprint" "Connector_JST:JST_SH_SM04B-SRSS-TB_1x04-1MP_P1.00mm_Horizontal" (id 2) (at 162.56 93.98 0)
+      (effects (font (size 1.27 1.27)) hide)
+    )
+    (property "Datasheet" "~" (id 3) (at 162.56 93.98 0)
+      (effects (font (size 1.27 1.27)) hide)
+    )
+    (pin "1")
+    (pin "2")
+    (pin "3")
+    (pin "4")
+  )
   (symbol (lib_id "keyboard_parts:KEYSW") (at 43.18 129.54 0) (mirror y) (unit 1)
     (in_bom yes) (on_board yes)
@@
       (reference "#PWR0121") (unit 1) (value "VCC") (footprint "")
     )
+    (path "/01b48b9a-0a9e-4863-aa93-97e7c72a5c2c"
+      (reference "#PWR0122") (unit 1) (value "GND") (footprint "")
+    )
     (path "/00000000-0000-0000-0000-00005c813d9c"
       (reference "C101") (unit 1) (value "1u") (footprint "Keeb_components:C_0805")
@@
       (reference "J2") (unit 1) (value "ISP") (footprint "Keeb_components:isp_standard")
     )
+    (path "/59536034-3f6c-43d8-85f3-720452bef88c"
+      (reference "J3") (unit 1) (value "UDB") (footprint "Connector_JST:JST_SH_SM04B-SRSS-TB_1x04-1MP_P1.00mm_Horizontal")
+    )
     (path "/00000000-0000-0000-0000-00005c891a9e"

Commit message: add proper jst
Parts:
- removed J3: UDB, Connector_JST:JST_SH_SM04B-SRSS-TB_1x04-1MP_P1.00mm_Horizontal, symbol Connector_Generic:Conn_01x04
- added J3: S5B-PH-K-S, Connector_JST:JST_PH_S5B-PH-K_1x05_P2.00mm_Horizontal, symbol Connector_Generic:Conn_01x05
Connections:
- net D+: now also J3.4 (Pin_4)
- net D-: now also J3.3 (Pin_3)
- net GND: now also J3.1 (Pin_1), J3.2 (Pin_2)
- net VUSB: now also J3.5 (Pin_5)
Changed lines of the file:
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@@
   (junction (at 152.4 162.56) (diameter 1.016) (color 0 0 0 0))
   (junction (at 152.4 184.15) (diameter 1.016) (color 0 0 0 0))
+  (junction (at 156.21 105.41) (diameter 1.016) (color 0 0 0 0))
   (junction (at 156.21 139.7) (diameter 1.016) (color 0 0 0 0))
   (junction (at 156.21 156.21) (diameter 1.016) (color 0 0 0 0))
@@
     (stroke (width 0) (type solid) (color 0 0 0 0))
   )
+  (wire (pts (xy 153.67 95.25) (xy 157.48 95.25))
+    (stroke (width 0) (type solid) (color 0 0 0 0))
+  )
+  (wire (pts (xy 153.67 102.87) (xy 156.21 102.87))
+    (stroke (width 0) (type solid) (color 0 0 0 0))
+  )
+  (wire (pts (xy 156.21 102.87) (xy 156.21 105.41))
+    (stroke (width 0) (type solid) (color 0 0 0 0))
+  )
+  (wire (pts (xy 156.21 105.41) (xy 153.67 105.41))
+    (stroke (width 0) (type solid) (color 0 0 0 0))
+  )
   (wire (pts (xy 156.21 129.54) (xy 156.21 130.81))
     (stroke (width 0) (type solid) (color 0 0 0 0))
@@
     (stroke (width 0) (type solid) (color 0 0 0 0))
   )
-  (wire (pts (xy 157.48 91.44) (xy 157.48 86.36))
+  (wire (pts (xy 157.48 95.25) (xy 157.48 86.36))
     (stroke (width 0) (type solid) (color 0 0 0 0))
   )
@@
     )
   )
-  (global_label "DIP1" (shape input) (at 154.94 69.85 90)
+  (global_label "D+" (shape input) (at 153.67 97.79 0)
     (effects (font (size 0.9906 0.9906)) (justify left))
-    (property "Intersheet References" "${INTERSHEET_REFS}" (id 0) (at 0 0 0)
+    (property "Intersheet References" "${INTERSHEET_REFS}" (id 0) (at 80.01 30.48 0)
       (effects (font (size 1.27 1.27)) hide)
     )
   )
-  (global_label "D-" (shape input) (at 157.48 93.98 180)
-    (effects (font (size 0.9906 0.9906)) (justify right))
-    (property "Intersheet References" "${INTERSHEET_REFS}" (id 0) (at 240.03 -58.42 0)
+  (global_label "D-" (shape input) (at 153.67 100.33 0)
+    (effects (font (size 0.9906 0.9906)) (justify left))
+    (property "Intersheet References" "${INTERSHEET_REFS}" (id 0) (at 80.01 30.48 0)
       (effects (font (size 1.27 1.27)) hide)
     )
   )
-  (global_label "D+" (shape input) (at 157.48 96.52 180)
-    (effects (font (size 0.9906 0.9906)) (justify right))
-    (property "Intersheet References" "${INTERSHEET_REFS}" (id 0) (at 240.03 -53.34 0)
+  (global_label "DIP1" (shape input) (at 154.94 69.85 90)
+    (effects (font (size 0.9906 0.9906)) (justify left))
+    (property "Intersheet References" "${INTERSHEET_REFS}" (id 0) (at 0 0 0)
       (effects (font (size 1.27 1.27)) hide)
     )
@@
     (pin "1")
   )
-  (symbol (lib_id "Power:GND") (at 157.48 66.04 180) (unit 1)
+  (symbol (lib_id "Power:GND") (at 156.21 105.41 90) (unit 1)
     (in_bom yes) (on_board yes)
-    (property "Reference" "#PWR0105" (id 0) (at 157.48 59.69 0)
+    (property "Reference" "#PWR0122" (id 0) (at 162.56 105.41 0)
       (effects (font (size 1.27 1.27)) hide)
     )
-    (property "Value" "GND" (id 1) (at 157.353 61.6458 0))
-    (property "Footprint" "" (id 2) (at 157.48 66.04 0)
+    (property "Value" "GND" (id 1) (at 160.6042 105.283 0))
+    (property "Footprint" "" (id 2) (at 156.21 105.41 0)
       (effects (font (size 1.27 1.27)) hide)
     )
-    (property "Datasheet" "" (id 3) (at 157.48 66.04 0)
+    (property "Datasheet" "" (id 3) (at 156.21 105.41 0)
       (effects (font (size 1.27 1.27)) hide)
     )
     (pin "1")
   )
-  (symbol (lib_id "power:GND") (at 157.48 99.06 0) (unit 1)
-    (in_bom yes) (on_board yes) (fields_autoplaced)
-    (property "Reference" "#PWR0122" (id 0) (at 157.48 105.41 0)
+  (symbol (lib_id "Power:GND") (at 157.48 66.04 180) (unit 1)
+    (in_bom yes) (on_board yes)
+    (property "Reference" "#PWR0105" (id 0) (at 157.48 59.69 0)
       (effects (font (size 1.27 1.27)) hide)
     )
-    (property "Value" "GND" (id 1) (at 157.48 104.14 0))
-    (property "Footprint" "" (id 2) (at 157.48 99.06 0)
+    (property "Value" "GND" (id 1) (at 157.353 61.6458 0))
+    (property "Footprint" "" (id 2) (at 157.48 66.04 0)
       (effects (font (size 1.27 1.27)) hide)
     )
-    (property "Datasheet" "" (id 3) (at 157.48 99.06 0)
+    (property "Datasheet" "" (id 3) (at 157.48 66.04 0)
       (effects (font (size 1.27 1.27)) hide)
     )
@@
     (pin "2")
   )
-  (symbol (lib_id "Connector_Generic:Conn_01x04") (at 162.56 93.98 0) (unit 1)
-    (in_bom yes) (on_board yes) (fields_autoplaced)
-    (property "Reference" "J3" (id 0) (at 165.1 93.9799 0)
-      (effects (font (size 1.27 1.27)) (justify left))
-    )
-    (property "Value" "UDB" (id 1) (at 165.1 96.5199 0)
-      (effects (font (size 1.27 1.27)) (justify left))
-    )
-    (property "Footprint" "Connector_JST:JST_SH_SM04B-SRSS-TB_1x04-1MP_P1.00mm_Horizontal" (id 2) (at 162.56 93.98 0)
-      (effects (font (size 1.27 1.27)) hide)
-    )
-    (property "Datasheet" "~" (id 3) (at 162.56 93.98 0)
-      (effects (font (size 1.27 1.27)) hide)
-    )
-    (pin "1")
-    (pin "2")
-    (pin "3")
-    (pin "4")
-  )
   (symbol (lib_id "keyboard_parts:KEYSW") (at 43.18 129.54 0) (mirror y) (unit 1)
     (in_bom yes) (on_board yes)
@@
     (pin "2")
   )
+  (symbol (lib_id "Connector_Generic:Conn_01x05") (at 148.59 100.33 180) (unit 1)
+    (in_bom yes) (on_board yes)
+    (property "Reference" "J3" (id 0) (at 150.6728 89.535 0))
+    (property "Value" "S5B-PH-K-S" (id 1) (at 150.6728 91.8464 0))
+    (property "Footprint" "Connector_JST:JST_PH_S5B-PH-K_1x05_P2.00mm_Horizontal" (id 2) (at 148.59 100.33 0)
+      (effects (font (size 1.27 1.27)) hide)
+    )
+    (property "Datasheet" "~" (id 3) (at 148.59 100.33 0)
+      (effects (font (size 1.27 1.27)) hide)
+    )
+    (pin "1")
+    (pin "2")
+    (pin "3")
+    (pin "4")
+    (pin "5")
+  )
   (symbol (lib_id "Connector_Generic:Conn_02x03_Odd_Even") (at 207.01 25.4 0) (unit 1)
     (in_bom yes) (on_board yes)
@@
       (reference "#PWR0121") (unit 1) (value "VCC") (footprint "")
     )
-    (path "/01b48b9a-0a9e-4863-aa93-97e7c72a5c2c"
+    (path "/bff7b0ab-2893-479e-96bb-531b5f5ed830"
       (reference "#PWR0122") (unit 1) (value "GND") (footprint "")
     )
@@
       (reference "J2") (unit 1) (value "ISP") (footprint "Keeb_components:isp_standard")
     )
-    (path "/59536034-3f6c-43d8-85f3-720452bef88c"
-      (reference "J3") (unit 1) (value "UDB") (footprint "Connector_JST:JST_SH_SM04B-SRSS-TB_1x04-1MP_P1.00mm_Horizontal")
+    (path "/a3459870-e1d4-48d2-ad62-18f0a5d398fd"
+      (reference "J3") (unit 1) (value "S5B-PH-K-S") (footprint "Connector_JST:JST_PH_S5B-PH-K_1x05_P2.00mm_Horizontal")
     )
     (path "/00000000-0000-0000-0000-00005c891a9e"
